File: pico-stretch2.kicad_pcb (KiCad board)
At the start: 4 copper layers, 82.1 x 21 mm, 66 parts, among them J2 Conn_01x03_Pin, J4 Conn_01x64_Castellated_Pads, U1 RP2350B_C42415655, U3 ME6217C33M5G, U4 W25Q128JVSIQTR, U5 RPI Radio Module 2, U6 ESP-PSRAM32, X1 ABM8-272-T3_C20625731

Commit message: Carry over pico-stretch review fixes
- U6 PSRAM is now APS6404L-3SQR (C5333729, 3.3 V); ESP-PSRAM32 is a 1.8 V part. Marked DNP, Exclude DNP on
- LCSC C1525 on C3/C4/C6 (the BOM rows had no part number)
- Silk ADC labels fixed (47A7..41A1); stray line breaks removed from "44A3" and "21"
- Courtyards on U1, USB1, X1, L1, D2, D3, Boot1, Reset1, PWR_LED1 and J4 (board and project libraries);
  tight pairs as built exempted by name in pico-stretch2.kicad_dru
- Stackup set to JLC04161H-7628
- Project copies of the symbol libraries the schematic uses (libs/, RPI_RMC20452T.kicad_sym, 15 pF in
  EasyEDA.kicad_sym); J2 model path on KICAD10_3DMODEL_DIR; stray power-symbol footprint fields cleared
- README: pins 60/61 fixed, optional-parts and ordering notes
Parts:
- U6: value ESP-PSRAM32 -> APS6404L-3SQR
Other:
- board text added: "41A1"
- board text added: "42A2"
- board text added: "43A3"
- board text added: "44A4"
- board text added: "45A5"
- board text added: "46A6"
- board text added: "47A7"
- board text removed: "41A6"
- board text removed: "42A5"
- board text removed: "43A4"
- board text removed: "44A3"
- board text removed: "45A2"
- board text removed: "46A1"
- board text removed: "47A0"
Changed lines of the file:
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@@
 			)
 			(layer "dielectric 1"
-				(type "core")
-				(thickness 0.48)
-				(material "FR4")
-				(epsilon_r 4.5)
+				(type "prepreg")
+				(thickness 0.2104)
+				(material "7628")
+				(epsilon_r 4.4)
 				(loss_tangent 0.02)
 			)
 			(layer "In1.Cu"
 				(type "copper")
-				(thickness 0.035)
+				(thickness 0.0152)
 			)
 			(layer "dielectric 2"
-				(type "prepreg")
-				(thickness 0.48)
+				(type "core")
+				(thickness 1.065)
 				(material "FR4")
-				(epsilon_r 4.5)
+				(epsilon_r 4.6)
 				(loss_tangent 0.02)
 			)
 			(layer "In2.Cu"
 				(type "copper")
-				(thickness 0.035)
+				(thickness 0.0152)
 			)
 			(layer "dielectric 3"
-				(type "core")
-				(thickness 0.48)
-				(material "FR4")
-				(epsilon_r 4.5)
+				(type "prepreg")
+				(thickness 0.2104)
+				(material "7628")
+				(epsilon_r 4.4)
 				(loss_tangent 0.02)
 			)
@@
 		)
 		(embedded_fonts no)
-		(model "${KICAD9_3DMODEL_DIR}/Connector_PinHeader_2.54mm.3dshapes/PinHeader_1x03_P2.54mm_Vertical.step"
+		(model "${KICAD10_3DMODEL_DIR}/Connector_PinHeader_2.54mm.3dshapes/PinHeader_1x03_P2.54mm_Vertical.step"
 			(offset
 				(xyz 0 0 0)
@@
 			(layer "F.SilkS")
 		)
+		(fp_rect
+			(start -2.9 -1.63)
+			(end 2.9 1.65)
+			(stroke
+				(width 0.05)
+				(type solid)
+			)
+			(fill no)
+			(layer "F.CrtYd")
+		)
 		(pad "1" smd rect
 			(at -2.199898 -1.099949)
@@
 			)
 		)
+		(property "LCSC" "C1525"
+			(at 0 0 0)
+			(layer "F.Fab")
+			(hide yes)
+			(effects
+				(font
+					(size 1 1)
+					(thickness 0.15)
+				)
+			)
+		)
 		(sheetname "/")
 		(sheetfile "pico-stretch2.kicad_sch")
@@
 			(layer "F.Fab")
 		)
+		(fp_rect
+			(start -1.09 -0.61)
+			(end 1.09 0.61)
+			(stroke
+				(width 0.05)
+				(type solid)
+			)
+			(fill no)
+			(layer "F.CrtYd")
+		)
 		(pad "1" smd rect
 			(at -0.5 0 180)
@@
 			(layer "F.Fab")
 		)
+		(fp_rect
+			(start -5.35 -5.35)
+			(end 5.35 5.35)
+			(stroke
+				(width 0.05)
+				(type solid)
+			)
+			(fill no)
+			(layer "F.CrtYd")
+		)
 		(pad "1" smd rect
 			(at -4.907544 -3.800102 90)
@@
 			(layer "F.Fab")
 		)
+		(fp_rect
+			(start -5.03 -3.03)
+			(end 5.03 3.38)
+			(stroke
+				(width 0.05)
+				(type solid)
+			)
+			(fill no)
+			(layer "F.CrtYd")
+		)
 		(pad "" np_thru_hole circle
 			(at -2.889891 -1.304928 270)
@@
 			(layer "F.Fab")
 		)
+		(fp_rect
+			(start -1.59 -0.86)
+			(end 1.5 0.85)
+			(stroke
+				(width 0.05)
+				(type solid)
+			)
+			(fill no)
+			(layer "F.CrtYd")
+		)
 		(pad "1" smd rect
 			(at -0.748997 0.000127 90)
@@
 			)
 		)
+		(property "LCSC" "C1525"
+			(at 0 0 270)
+			(layer "F.Fab")
+			(hide yes)
+			(effects
+				(font
+					(size 1 1)
+					(thickness 0.15)
+				)
+			)
+		)
 		(sheetname "/")
 		(sheetfile "pico-stretch2.kicad_sch")
@@
 			(layer "F.Fab")
 		)
+		(fp_rect
+			(start -2.36 -1.78)
+			(end 2.13 2.01)
+			(stroke
+				(width 0.05)
+				(type solid)
+			)
+			(fill no)
+			(layer "F.CrtYd")
+		)
 		(pad "1" smd rect
 			(at -1.100076 0.850013 90)
@@
 			(layer "F.Fab")
 		)
+		(fp_rect
+			(start -1.6 -1.33)
+			(end 1.6 0.9)
+			(stroke
+				(width 0.05)
+				(type solid)
+			)
+			(fill no)
+			(layer "F.CrtYd")
+		)
 		(pad "1" smd rect
 			(at -1 0 270)
@@
 			)
 		)
+		(fp_rect
+			(start -0.95 -2.56)
+			(end 79.69 0.95)
+			(stroke
+				(width 0.05)
+				(type solid)
+			)
+			(fill no)
+			(layer "F.CrtYd")
+		)
+		(fp_rect
+			(start -0.95 16.82)
+			(end 79.69 20.34)
+			(stroke
+				(width 0.05)
+				(type solid)
+			)
+			(fill no)
+			(layer "F.CrtYd")
+		)
 		(pad "1" thru_hole oval
 			(at 0 17.78 180)
@@
 			)
 		)
+		(property "LCSC" "C1525"
+			(at 0 0 0)
+			(layer "F.Fab")
+			(hide yes)
+			(effects
+				(font
+					(size 1 1)
+					(thickness 0.15)
+				)
+			)
+		)
 		(sheetname "/")
 		(sheetfile "pico-stretch2.kicad_sch")
@@
 			(layer "F.SilkS")
 		)
+		(fp_rect
+			(start -2.9 -1.63)
+			(end 2.9 1.65)
+			(stroke
+				(width 0.05)
+				(type solid)
+			)
+			(fill no)
+			(layer "F.CrtYd")
+		)
 		(pad "1" smd rect
 			(at -2.199898 -1.099949 180)
@@
 			(layer "F.Fab")
 		)
+		(fp_rect
+			(start -1.09 -0.61)
+			(end 1.09 0.61)
+			(stroke
+				(width 0.05)
+				(type solid)
+			)
+			(fill no)
+			(layer "F.CrtYd")
+		)
 		(pad "1" smd rect
 			(at -0.5 0)
@@
 			)
 		)
-		(property "Value" "ESP-PSRAM32"
+		(property "Value" "APS6404L-3SQR"
 			(at 0 3.4 0)
 			(layer "F.Fab")
@@
 			)
 		)
-		(property "Datasheet" "https://www.espressif.com/sites/default/files/documentation/esp-psram32_datasheet_en.pdf"
+		(property "Datasheet" "https://www.lcsc.com/product-detail/C5333729.html"
 			(at 0 0 0)
 			(layer "F.Fab")
@@
 			)
 		)
-		(property "Description" "32 Mbit serial pseudo SRAM device organized as 4Mx8 bits, 1.8 VCC, SOIC8 (SOP8)"
+		(property "Description" "64 Mbit QSPI PSRAM, 2.7-3.6 V, SOP-8 150 mil (AP Memory APS6404L-3SQR-SN). Optional, not fitted."
 			(at 0 0 0)
 			(layer "F.Fab")
@@
 		)
 		(property ki_fp_filters "SOIC*3.9x4.9mm?P1.27mm*")
+		(property "LCSC" "C5333729"
+			(at 0 0 0)
+			(layer "F.Fab")
+			(hide yes)
+			(effects
+				(font
+					(size 1 1)
+					(thickness 0.15)
+				)
+			)
+		)
 		(sheetname "/")
 		(sheetfile "pico-stretch2.kicad_sch")
@@
 			)
 		)
-		(attr smd)
+		(attr smd dnp)
 		(duplicate_pad_numbers_are_jumpers no)
 		(fp_line
@@
 		)
 	)
-	(gr_text "41A6"
+	(gr_text "41A1"
 		(at 175.38 94.67 0)
 		(layer "F.SilkS")
@@
 		)
 	)
-	(gr_text "21\n"
+	(gr_text "21"
 		(at 144.22 95.18 90)
 		(layer "F.SilkS")
@@
 		)
 	)
-	(gr_text "47A0"
+	(gr_text "47A7"
 		(at 162.03 96.67 90)
 		(layer "F.SilkS")
@@
 		)
 	)
-	(gr_text "46A1"
+	(gr_text "46A6"
 		(at 164.59 96.69 90)
 		(layer "F.SilkS")
@@
 		)
 	)
-	(gr_text "45A2"
+	(gr_text "45A5"
 		(at 167.17 96.64 90)
 		(layer "F.SilkS")
@@
 		)
 	)
-	(gr_text "44A3\n"
+	(gr_text "44A4"
 		(at 169.75 96.57 90)
 		(layer "F.SilkS")
@@
 		)
 	)
-	(gr_text "43A4"
+	(gr_text "43A3"
 		(at 172.25 96.69 90)
 		(layer "F.SilkS")
@@
 		)
 	)
-	(gr_text "42A5"
+	(gr_text "42A2"
 		(at 174.799678 96.64 90)
 		(layer "F.SilkS")
