File: pico-stretch2.kicad_sch (KiCad schematic)
At the start: 64 parts, among them J2 Conn_01x03_Pin, J4 Conn_01x64_Castellated_Pads, U1 RP2350B_C42415655, U3 ME6217C33M5G, U4 W25Q128JVSIQTR, U5 RPI Radio Module 2, U6 ESP-PSRAM32, X1 ABM8-272-T3_C20625731

Commit message: Carry over pico-stretch review fixes
- U6 PSRAM is now APS6404L-3SQR (C5333729, 3.3 V); ESP-PSRAM32 is a 1.8 V part. Marked DNP, Exclude DNP on
- LCSC C1525 on C3/C4/C6 (the BOM rows had no part number)
- Silk ADC labels fixed (47A7..41A1); stray line breaks removed from "44A3" and "21"
- Courtyards on U1, USB1, X1, L1, D2, D3, Boot1, Reset1, PWR_LED1 and J4 (board and project libraries);
  tight pairs as built exempted by name in pico-stretch2.kicad_dru
- Stackup set to JLC04161H-7628
- Project copies of the symbol libraries the schematic uses (libs/, RPI_RMC20452T.kicad_sym, 15 pF in
  EasyEDA.kicad_sym); J2 model path on KICAD10_3DMODEL_DIR; stray power-symbol footprint fields cleared
- README: pins 60/61 fixed, optional-parts and ordering notes
Parts:
- C3, C4, C6: LCSC (none) -> C1525
- U6: value ESP-PSRAM32 -> APS6404L-3SQR; LCSC (none) -> C5333729; now not fitted
Changed lines of the file:
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@@
 			)
 		)
+		(property "LCSC" "C1525"
+			(at 209.55 87.63 0)
+			(hide yes)
+			(show_name no)
+			(do_not_autoplace no)
+			(effects
+				(font
+					(size 1.27 1.27)
+				)
+			)
+		)
 		(pin "2"
 		)
@@
 			)
 		)
-		(property "Footprint" "RP2350 Dev Board:"
+		(property "Footprint" ""
 			(at 116.84 295.91 0)
 			(hide yes)
@@
 			)
 		)
+		(property "LCSC" "C1525"
+			(at 214.63 87.63 0)
+			(hide yes)
+			(show_name no)
+			(do_not_autoplace no)
+			(effects
+				(font
+					(size 1.27 1.27)
+				)
+			)
+		)
 		(pin "2"
 		)
@@
 			)
 		)
-		(property "Footprint" "RP2350 Dev Board:"
+		(property "Footprint" ""
 			(at 82.55 116.84 0)
 			(hide yes)
@@
 			)
 		)
-		(property "Footprint" "RP2350 Dev Board:"
+		(property "Footprint" ""
 			(at 242.57 257.81 0)
 			(hide yes)
@@
 		(on_board yes)
 		(in_pos_files yes)
-		(dnp no)
+		(dnp yes)
 		(fields_autoplaced yes)
 		(property "Reference" "U6"
@@
 			)
 		)
-		(property "Value" "ESP-PSRAM32"
+		(property "Value" "APS6404L-3SQR"
 			(at 54.61 298.45 90)
 			(show_name no)
@@
 			)
 		)
-		(property "Datasheet" "https://www.espressif.com/sites/default/files/documentation/esp-psram32_datasheet_en.pdf"
+		(property "Datasheet" "https://www.lcsc.com/product-detail/C5333729.html"
 			(at 67.31 298.45 0)
 			(hide yes)
@@
 			)
 		)
-		(property "Description" "32 Mbit serial pseudo SRAM device organized as 4Mx8 bits, 1.8 VCC, SOIC8 (SOP8)"
+		(property "Description" "64 Mbit QSPI PSRAM, 2.7-3.6 V, SOP-8 150 mil (AP Memory APS6404L-3SQR-SN). Optional, not fitted."
+			(at 54.61 308.61 0)
+			(hide yes)
+			(show_name no)
+			(do_not_autoplace no)
+			(effects
+				(font
+					(size 1.27 1.27)
+				)
+			)
+		)
+		(property "LCSC" "C5333729"
 			(at 54.61 308.61 0)
 			(hide yes)
@@
 			)
 		)
-		(property "Footprint" "RP2350 Dev Board:"
+		(property "Footprint" ""
 			(at 195.58 295.91 0)
 			(hide yes)
@@
 			(at 219.71 87.63 0)
 			(hide yes)
+			(show_name no)
+			(do_not_autoplace no)
+			(effects
+				(font
+					(size 1.27 1.27)
+				)
+			)
+		)
+		(property "LCSC" "C1525"
+			(at 219.71 87.63 0)
+			(hide yes)

Commit message: USB test pads, PSRAM CS on GPIO0 or GPIO47, back-side pin labels
- TP3 (USB D-) and TP4 (USB D+) on the back, connector side of R2/R3; new via in D2's signal pad for D-
- JP4 (back, beside U6) selects GPIO47 as the PSRAM chip select; JP1 still selects GPIO0. GPIO47 reaches
  JP4 on a 0.15 mm Inner2 track from castellated pad 44 along y 94.05 (back-layer traces only cross it,
  every via 0.42 mm or more away) and one via; JP4 sits at the PSRAM end so an open JP4 leaves no stub
- Every castellated pad labelled on the back (same text as the front); D-/D+ beside the test pads;
  jumper note moved off TP4 and rewritten for JP4; back logo moved down 2.9 mm to clear the labels
- README: PSRAM jumper choice, back-side notes
Parts:
- added JP4: SolderJumper_2_Open, Jumper:SolderJumper-2_P1.3mm_Open_Pad1.0x1.5mm, symbol Jumper:SolderJumper_2_Open
- added TP3, TP4: TestPoint, TestPoint:TestPoint_Pad_1.0x1.0mm, symbol Connector:TestPoint
Connections:
- net GPIO47/ADC7: now also JP4.2 (B)
- net USB2_D+: now also TP4.1
- net USB2_D-: now also TP3.1
- net at JP1.1 (A), R14.1, U6.1 (~{CE}): now also JP4.1 (A)

Commit message: Apply design review fixes and add re-review
Review 1 fixes (scripts/review_fixes.py, rebuilds from 54e971f):
- C9/C15 to 0402 C1525, R14 to 1k, C40 to 0603 10 uF with via-in-pad
- D3 in line on USB D+, C39 flipped to share D3 ground via
- C13 moved 0.05 mm clear of U1 pin 50
- Extended In1 VREG_LX cut-out, J4 pads 29-36 clipped
- U5 DNP with no paste, silkscreen fixes, named courtyard pairs
- VBUS TVS tried and removed

DESIGN_REVIEW_2.md and review2/ hold the re-review and its pack.
Parts:
- C15, C9: LCSC C14663 -> C1525; LCSC Part Name 100nF ±10% 50V -> 100nF ±10% 16V; Manufacturer YAGEO(国巨) -> SAMSUNG(三星); Manufacturer Part CC0603KRX7R9BB104 -> CL05B104KO5NNNC; Temperature Coefficient X7R -> (none); Voltage Rating 50V -> (none)
- C40: value CL05A106MQ5NUNC -> 10uF; footprint Capacitor_SMD:C_0402_1005Metric -> Capacitor_SMD:C_0603_1608Metric; Attrition Qty (none) -> 10; Capacitance (none) -> 10uF; Category (none) -> Capacitors,Multilayer Ceramic Capacitors MLCC - SMD/SMT; Class (none) -> Basic Component; LCSC C15525 -> C19702; Manufacturer Part CL05A106MQ5NUNC -> (none); Minimum Qty (none) -> 20; Part (none) -> CL10A106KP8NNNC; Price (none) -> 0.009USD; Process (none) -> SMT; Stock (none) -> 11716291; Temperature Coefficient (none) -> X5R; Tolerance (none) -> ±10%; Voltage Rated (none) -> 10V
- R14: value 10kΩ -> 1kΩ; LCSC C25744 -> C11702; Minimum Qty 5 -> 20; Part 0402WGF1002TCE -> 0402WGF1001TCE; Resistance 10kΩ -> 1kΩ; Stock 18633144 -> 12206505
- U5: now not fitted
Changed lines of the file:
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@@
 			)
 		)
-		(property "Value" "CL05A106MQ5NUNC"
+		(property "Value" "10uF"
 			(at 187.96 304.7999 90)
 			(hide yes)
@@
 			)
 		)
-		(property "Footprint" "Capacitor_SMD:C_0402_1005Metric"
+		(property "Footprint" "Capacitor_SMD:C_0603_1608Metric"
 			(at 184.15 303.53 0)
 			(hide yes)
@@
 			)
 		)
-		(property "Datasheet" "https://www.lcsc.com/datasheet/lcsc_datasheet_2208231630_Samsung-Electro-Mechanics-CL05A106MQ5NUNC_C15525.pdf"
+		(property "Datasheet" "https://www.lcsc.com/datasheet/lcsc_datasheet_2304140030_Samsung-Electro-Mechanics-CL10A106KP8NNNC_C19702.pdf"
 			(at 184.15 303.53 0)
 			(hide yes)
@@
 			)
 		)
-		(property "Description" "10uF 6.3V X5R ±20% 0402 Multilayer Ceramic Capacitors MLCC - SMD/SMT ROHS"
+		(property "Description" "10V 10uF X5R ±10% 0603 Multilayer Ceramic Capacitors MLCC - SMD/SMT ROHS"
 			(at 184.15 303.53 0)
 			(hide yes)
@@
 			)
 		)
-		(property "LCSC" "C15525"
+		(property "LCSC" "C19702"
 			(at 184.15 303.53 0)
 			(hide yes)
@@
 			)
 		)
-		(property "Manufacturer Part" "CL05A106MQ5NUNC"
+		(property "Stock" "11716291"
+			(at 184.15 303.53 0)
+			(hide yes)
+			(show_name no)
+			(do_not_autoplace no)
+			(effects
+				(font
+					(size 1.27 1.27)
+				)
+			)
+		)
+		(property "Price" "0.009USD"
+			(at 184.15 303.53 0)
+			(hide yes)
+			(show_name no)
+			(do_not_autoplace no)
+			(effects
+				(font
+					(size 1.27 1.27)
+				)
+			)
+		)
+		(property "Process" "SMT"
+			(at 184.15 303.53 0)
+			(hide yes)
+			(show_name no)
+			(do_not_autoplace no)
+			(effects
+				(font
+					(size 1.27 1.27)
+				)
+			)
+		)
+		(property "Minimum Qty" "20"
+			(at 184.15 303.53 0)
+			(hide yes)
+			(show_name no)
+			(do_not_autoplace no)
+			(effects
+				(font
+					(size 1.27 1.27)
+				)
+			)
+		)
+		(property "Attrition Qty" "10"
+			(at 184.15 303.53 0)
+			(hide yes)
+			(show_name no)
+			(do_not_autoplace no)
+			(effects
+				(font
+					(size 1.27 1.27)
+				)
+			)
+		)
+		(property "Class" "Basic Component"
+			(at 184.15 303.53 0)
+			(hide yes)
+			(show_name no)
+			(do_not_autoplace no)
+			(effects
+				(font
+					(size 1.27 1.27)
+				)
+			)
+		)
+		(property "Category" "Capacitors,Multilayer Ceramic Capacitors MLCC - SMD/SMT"
+			(at 184.15 303.53 0)
+			(hide yes)
+			(show_name no)
+			(do_not_autoplace no)
+			(effects
+				(font
+					(size 1.27 1.27)
+				)
+			)
+		)
+		(property "Part" "CL10A106KP8NNNC"
+			(at 184.15 303.53 0)
+			(hide yes)
+			(show_name no)
+			(do_not_autoplace no)
+			(effects
+				(font
+					(size 1.27 1.27)
+				)
+			)
+		)
+		(property "Voltage Rated" "10V"
+			(at 184.15 303.53 0)
+			(hide yes)
+			(show_name no)
+			(do_not_autoplace no)
+			(effects
+				(font
+					(size 1.27 1.27)
+				)
+			)
+		)
+		(property "Tolerance" "±10%"
+			(at 184.15 303.53 0)
+			(hide yes)
+			(show_name no)
+			(do_not_autoplace no)
+			(effects
+				(font
+					(size 1.27 1.27)
+				)
+			)
+		)
+		(property "Capacitance" "10uF"
+			(at 184.15 303.53 0)
+			(hide yes)
+			(show_name no)
+			(do_not_autoplace no)
+			(effects
+				(font
+					(size 1.27 1.27)
+				)
+			)
+		)
+		(property "Temperature Coefficient" "X5R"
 			(at 184.15 303.53 0)
 			(hide yes)
@@
 		(on_board yes)
 		(in_pos_files yes)
-		(dnp no)
+		(dnp yes)
 		(fields_autoplaced yes)
 		(property "Reference" "U5"
@@
 			)
 		)
-		(property "Datasheet" "https://atta.szlcsc.com/upload/public/pdf/source/20180910/C282072_33301C7F631E79921B82A8DAC6BCC5B3.pdf"
+		(property "Datasheet" "https://atta.szlcsc.com/upload/public/pdf/source/20160218/1457707763339.pdf"
 			(at 128.27 219.71 0)
 			(hide yes)
@@
 			)
 		)
-		(property "Description" "Capacitance:100nF Tolerance:±10% Tolerance:±10% Voltage Rating:50V Temperature Coefficient:X7R"
+		(property "Description" "Capacitance: Tolerance:±10% Tolerance:±10% Voltage Rated: Temperature Coefficient:"
 			(at 128.27 219.71 0)
 			(hide yes)
@@
 			)
 		)
-		(property "Manufacturer Part" "CC0603KRX7R9BB104"
+		(property "Manufacturer Part" "CL05B104KO5NNNC"
 			(at 128.27 219.71 0)
 			(hide yes)
@@
 			)
 		)
-		(property "Manufacturer" "YAGEO(国巨)"
+		(property "Manufacturer" "SAMSUNG(三星)"
 			(at 128.27 219.71 0)
 			(hide yes)
@@
 			)
 		)
-		(property "LCSC Part Name" "100nF ±10% 50V"
-			(at 128.27 219.71 0)
-			(hide yes)
-			(show_name no)
-			(do_not_autoplace no)
-			(effects
-				(font
-					(size 1.27 1.27)
-				)
-			)
-		)
-		(property "Temperature Coefficient" "X7R"
-			(at 125.73 226.06 0)
-			(hide yes)
-			(show_name no)
-			(do_not_autoplace no)
-			(effects
-				(font
-					(size 1.27 1.27)
-				)
-				(justify left bottom)
-			)
-		)
-		(property "Voltage Rating" "50V"
+		(property "LCSC Part Name" "100nF ±10% 16V"
 			(at 128.27 219.71 0)
 			(hide yes)
@@
 					(size 1.27 1.27)
 				)
-				(justify left bottom)
 			)
 		)
-		(property "LCSC" "C14663"
+		(property "LCSC" "C1525"
 			(at 128.27 219.71 0)
 			(hide yes)
@@
 			)
 		)
-		(property "Datasheet" "https://atta.szlcsc.com/upload/public/pdf/source/20180910/C282072_33301C7F631E79921B82A8DAC6BCC5B3.pdf"
+		(property "Datasheet" "https://atta.szlcsc.com/upload/public/pdf/source/20160218/1457707763339.pdf"
 			(at 204.47 87.63 0)
 			(hide yes)
@@
 			)
 		)
-		(property "Description" "Capacitance:100nF Tolerance:±10% Tolerance:±10% Voltage Rating:50V Temperature Coefficient:X7R"
+		(property "Description" "Capacitance: Tolerance:±10% Tolerance:±10% Voltage Rated: Temperature Coefficient:"
 			(at 204.47 87.63 90)
 			(hide yes)
@@
 			)
 		)
-		(property "Manufacturer Part" "CC0603KRX7R9BB104"
+		(property "Manufacturer Part" "CL05B104KO5NNNC"
 			(at 204.47 87.63 0)
 			(hide yes)
@@
 			)
 		)
-		(property "Manufacturer" "YAGEO(国巨)"
+		(property "Manufacturer" "SAMSUNG(三星)"
 			(at 204.47 87.63 0)
 			(hide yes)
@@
 			)
 		)
-		(property "LCSC Part Name" "100nF ±10% 50V"
+		(property "LCSC Part Name" "100nF ±10% 16V"
 			(at 204.47 87.63 0)
 			(hide yes)
@@
 			)
 		)
-		(property "Temperature Coefficient" "X7R"
-			(at 212.09 90.17 90)
-			(hide yes)
-			(show_name no)
-			(do_not_autoplace no)
-			(effects
-				(font
-					(size 1.27 1.27)
-				)
-				(justify left bottom)
-			)
-		)
-		(property "Voltage Rating" "50V"
-			(at 204.47 87.63 90)
-			(hide yes)
-			(show_name no)
-			(do_not_autoplace no)
-			(effects
-				(font
-					(size 1.27 1.27)
-				)
-				(justify left bottom)
-			)
-		)
-		(property "LCSC" "C14663"
+		(property "LCSC" "C1525"
 			(at 204.47 87.63 90)
 			(hide yes)
@@
 			)
 		)
-		(property "Value" "10kΩ"
+		(property "Value" "1kΩ"
 			(at 46.99 294.64 90)
 			(show_name no)
@@
 			)
 		)
-		(property "Datasheet" "https://www.lcsc.com/datasheet/lcsc_datasheet_2411221126_UNI-ROYAL-Uniroyal-Elec-0402WGF1002TCE_C25744.pdf"
+		(property "Datasheet" "https://www.lcsc.com/datasheet/lcsc_datasheet_2206010216_UNI-ROYAL-Uniroyal-Elec-0402WGF1001TCE_C11702.pdf"
 			(at 46.99 294.64 0)
 			(hide yes)
@@
 			)
 		)
-		(property "Description" "62.5mW Thick Film Resistors 50V ±100ppm/°C ±1% 10kΩ 0402 Chip Resistor - Surface Mount ROHS"
+		(property "Description" "62.5mW Thick Film Resistors 50V ±100ppm/°C ±1% 1kΩ 0402 Chip Resistor - Surface Mount ROHS"
 			(at 46.99 294.64 0)
 			(hide yes)
@@
 			)
 		)
-		(property "LCSC" "C25744"
+		(property "LCSC" "C11702"
 			(at 46.99 294.64 0)
 			(hide yes)
@@
 			)
 		)
-		(property "Stock" "18633144"
+		(property "Stock" "12206505"
 			(at 46.99 294.64 0)
 			(hide yes)
@@
 			)
 		)
-		(property "Minimum Qty" "5"
+		(property "Minimum Qty" "20"
 			(at 46.99 294.64 0)
 			(hide yes)
@@
 			)
 		)
-		(property "Part" "0402WGF1002TCE"
+		(property "Part" "0402WGF1001TCE"
 			(at 46.99 294.64 0)
 			(hide yes)
@@
 			)
 		)
-		(property "Resistance" "10kΩ"
+		(property "Resistance" "1kΩ"
 			(at 46.99 294.64 0)
 			(hide yes)

Commit message: Design review 3 fixes and Pico-footprint USB test pads
Review 3 (DESIGN_REVIEW_3.md, scripts/review3_fixes.py, from 1d4354a):
- 87 vias 0.4/0.2 -> 0.45/0.2 (JLC's free via); Default net class and
  DRC minimum via 0.45 mm; 0.45 mm via-to-plated-hole rule, hole_to_hole
  an error
- VREG_LX track 0.18 mm beside C10/C12 (JLC 0.1 mm pad-to-track)
- C2/C5 values swapped: 4.7 uF on DVDD pin 32, the pin furthest from
  the regulator (RP2350 datasheet 6.1.3)
- C9, RUN and GPIO47 vias moved off / into their own pads

USB test pads at the Pico 2's TP1-TP3 positions (scripts/pico_testpads.py),
so the board can be hot-plate soldered onto a Pico SMT footprint:
- TP3 (D-), TP4 (D+) and new TP5 (GND) on 1.5 x 1.5 mm R0.3 pads
  (Custom:TestPoint_Pad_1.5x1.5mm_R0.3mm), one new B.Cu stub each
- README: test pads and soldering onto a Pico footprint

review3/ holds the analysis packs, reviewer reports and via scripts.
production/ is still the pre-review output: regenerate before ordering.
Parts:
- added TP5: TestPoint, Custom:TestPoint_Pad_1.5x1.5mm_R0.3mm, symbol Connector:TestPoint
- C2: value 100nF -> 4.7uF; LCSC C1525 -> C23733; LCSC Part Name 100nF ±10% 16V -> (none); Manufacturer SAMSUNG(三星) -> Samsung Electro-Mechanics; Manufacturer Part CL05B104KO5NNNC -> CL05A475MP5NRNC; Supplier LCSC -> (none); Supplier Part C1525 -> (none)
- C5: value 4.7uF -> 100nF; LCSC C23733 -> C1525; LCSC Part Name (none) -> 100nF ±10% 16V; Manufacturer Samsung Electro-Mechanics -> SAMSUNG(三星); Manufacturer Part CL05A475MP5NRNC -> CL05B104KO5NNNC; Supplier (none) -> LCSC; Supplier Part (none) -> C1525
- TP3, TP4: footprint TestPoint:TestPoint_Pad_1.0x1.0mm -> Custom:TestPoint_Pad_1.5x1.5mm_R0.3mm
Connections:
- net GND: now also TP5.1
Changed lines of the file:
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@@
 		)
 	)
+	(wire
+		(pts
+			(xy 298.45 236.22) (xy 298.45 241.3)
+		)
+		(stroke
+			(width 0)
+			(type default)
+		)
+	)
 	(image
 		(at 412.75 153.67)
@@
 			)
 		)
-		(property "Value" "4.7uF"
+		(property "Value" "100nF"
 			(at 128.778 84.836 0)
 			(show_name no)
@@
 			)
 		)
-		(property "Datasheet" "https://www.lcsc.com/datasheet/lcsc_datasheet_2304140030_Samsung-Electro-Mechanics-CL05A475MP5NRNC_C23733.pdf"
+		(property "Datasheet" "https://atta.szlcsc.com/upload/public/pdf/source/20160218/1457707763339.pdf"
 			(at 127 83.82 0)
 			(hide yes)
@@
 			)
 		)
-		(property "Description" "10V 4.7uF X5R ±20% 0402 Multilayer Ceramic Capacitors MLCC - SMD/SMT ROHS"
+		(property "Description" "Capacitance: Tolerance:±10% Tolerance:±10% Voltage Rated: Temperature Coefficient:"
 			(at 127 83.82 0)
 			(hide yes)
@@
 			)
 		)
-		(property "LCSC" "C23733"
+		(property "LCSC" "C1525"
 			(at 127 83.82 0)
 			(hide yes)
@@
 			)
 		)
-		(property "Manufacturer" "Samsung Electro-Mechanics"
+		(property "Manufacturer" "SAMSUNG(三星)"
 			(at 127 83.82 0)
 			(hide yes)
@@
 			)
 		)
-		(property "Manufacturer Part" "CL05A475MP5NRNC"
+		(property "Manufacturer Part" "CL05B104KO5NNNC"
+			(at 127 83.82 0)
+			(hide yes)
+			(show_name no)
+			(do_not_autoplace no)
+			(effects
+				(font
+					(size 1.27 1.27)
+				)
+			)
+		)
+		(property "Supplier Part" "C1525"
+			(at 127 83.82 0)
+			(hide yes)
+			(show_name no)
+			(do_not_autoplace no)
+			(effects
+				(font
+					(size 1.27 1.27)
+				)
+			)
+		)
+		(property "Supplier" "LCSC"
+			(at 127 83.82 0)
+			(hide yes)
+			(show_name no)
+			(do_not_autoplace no)
+			(effects
+				(font
+					(size 1.27 1.27)
+				)
+			)
+		)
+		(property "LCSC Part Name" "100nF ±10% 16V"
 			(at 127 83.82 0)
 			(hide yes)
@@
 			)
 		)
-		(property "Value" "100nF"
+		(property "Value" "4.7uF"
 			(at 135.636 90.17 90)
 			(show_name no)
@@
 			)
 		)
-		(property "Datasheet" "https://atta.szlcsc.com/upload/public/pdf/source/20160218/1457707763339.pdf"
+		(property "Datasheet" "https://www.lcsc.com/datasheet/lcsc_datasheet_2304140030_Samsung-Electro-Mechanics-CL05A475MP5NRNC_C23733.pdf"
 			(at 133.35 83.82 0)
 			(hide yes)
@@
 			)
 		)
-		(property "Description" "Capacitance: Tolerance:±10% Tolerance:±10% Voltage Rated: Temperature Coefficient:"
+		(property "Description" "10V 4.7uF X5R ±20% 0402 Multilayer Ceramic Capacitors MLCC - SMD/SMT ROHS"
 			(at 133.35 83.82 90)
 			(hide yes)
@@
 			)
 		)
-		(property "Manufacturer Part" "CL05B104KO5NNNC"
-			(at 133.35 83.82 0)
-			(hide yes)
-			(show_name no)
-			(do_not_autoplace no)
-			(effects
-				(font
-					(size 1.27 1.27)
-				)
-			)
-		)
-		(property "Manufacturer" "SAMSUNG(三星)"
-			(at 133.35 83.82 0)
-			(hide yes)
-			(show_name no)
-			(do_not_autoplace no)
-			(effects
-				(font
-					(size 1.27 1.27)
-				)
-			)
-		)
-		(property "Supplier Part" "C1525"
-			(at 133.35 83.82 0)
-			(hide yes)
-			(show_name no)
-			(do_not_autoplace no)
-			(effects
-				(font
-					(size 1.27 1.27)
-				)
-			)
-		)
-		(property "Supplier" "LCSC"
+		(property "Manufacturer Part" "CL05A475MP5NRNC"
 			(at 133.35 83.82 0)
 			(hide yes)
@@
 			)
 		)
-		(property "LCSC Part Name" "100nF ±10% 16V"
+		(property "Manufacturer" "Samsung Electro-Mechanics"
 			(at 133.35 83.82 0)
 			(hide yes)
@@
 			)
 		)
-		(property "LCSC" "C1525"
+		(property "LCSC" "C23733"
 			(at 133.35 83.82 90)
 			(hide yes)
@@
 			)
 		)
-		(property "Footprint" "TestPoint:TestPoint_Pad_1.0x1.0mm"
+		(property "Footprint" "Custom:TestPoint_Pad_1.5x1.5mm_R0.3mm"
 			(at 290.83 236.22 0)
 			(hide yes)
@@
 			)
 		)
-		(property "Footprint" "TestPoint:TestPoint_Pad_1.0x1.0mm"
+		(property "Footprint" "Custom:TestPoint_Pad_1.5x1.5mm_R0.3mm"
 			(at 290.83 248.92 0)
 			(hide yes)
@@
 					(unit 1)
 				)
+			)
+		)
+	)
+	(symbol
+		(lib_id "Connector:TestPoint")
+		(at 298.45 236.22 0)
+		(unit 1)
+		(body_style 1)
+		(exclude_from_sim no)
+		(in_bom yes)
+		(on_board yes)
+		(in_pos_files yes)
+		(dnp no)
+		(property "Reference" "TP5"
+			(at 298.45 229.362 0)
+			(show_name no)
+			(do_not_autoplace no)
+			(effects
+				(font
+					(size 1.27 1.27)
+				)
+			)
+		)
+		(property "Value" "TestPoint"
+			(at 298.45 231.14 0)
+			(show_name no)
+			(do_not_autoplace no)
+			(effects
+				(font
+					(size 1.27 1.27)
+				)
+			)
+		)
+		(property "Footprint" "Custom:TestPoint_Pad_1.5x1.5mm_R0.3mm"
+			(at 303.53 236.22 0)
+			(hide yes)
+			(show_name no)
+			(do_not_autoplace no)
+			(effects
+				(font
+					(size 1.27 1.27)
+				)
+			)
+		)
+		(property "Datasheet" ""
+			(at 303.53 236.22 0)
+			(hide yes)
+			(show_name no)
+			(do_not_autoplace no)
+			(effects
+				(font
+					(size 1.27 1.27)
+				)
+			)
+		)
+		(property "Description" "test point"
+			(at 298.45 236.22 0)
+			(hide yes)
+			(show_name no)
+			(do_not_autoplace no)
+			(effects
+				(font
+					(size 1.27 1.27)
+				)
+			)
+		)
+		(pin "1"
+		)
+		(instances
+			(project "pico-stretch2"
+				(path "/879934c2-924b-48fd-aecd-6699a94a302d"
+					(reference "TP5")
+					(unit 1)
+				)
+			)
+		)
+	)
+	(symbol
+		(lib_id "power:GND")
+		(at 298.45 241.3 0)
+		(unit 1)
+		(body_style 1)
+		(exclude_from_sim no)
+		(in_bom no)
+		(on_board no)
+		(in_pos_files yes)
+		(dnp no)
+		(property "Reference" "#PWR001"
+			(at 298.45 247.65 0)
+			(hide yes)
+			(show_name no)
+			(do_not_autoplace no)
+			(effects
+				(font
+					(size 1.27 1.27)
+				)
+			)
+		)
+		(property "Value" "GND"
+			(at 298.45 245.11 0)
+			(show_name no)
+			(do_not_autoplace no)
+			(effects
+				(font
+					(size 1.27 1.27)
+				)
+			)
+		)
+		(property "Footprint" ""
+			(at 298.45 241.3 0)
+			(hide yes)
+			(show_name no)
+			(do_not_autoplace no)
+			(effects
+				(font
+					(size 1.27 1.27)
+				)
+			)
+		)
+		(property "Datasheet" ""
+			(at 298.45 241.3 0)
+			(hide yes)
+			(show_name no)
+			(do_not_autoplace no)
+			(effects
+				(font
+					(size 1.27 1.27)
+				)
+			)
+		)
+		(property "Description" "Power symbol creates a global label with name \"GND\" , ground"
+			(at 298.45 241.3 0)
+			(hide yes)
+			(show_name no)
+			(do_not_autoplace no)
+			(effects
+				(font
+					(size 1.27 1.27)
+				)
+			)
+		)
+		(pin "1"
+		)
+		(instances
+			(project "pico-stretch2"
+				(path "/879934c2-924b-48fd-aecd-6699a94a302d"
+					(reference "#PWR001")
+					(unit 1)
+				)
