File: pico-stretch2.kicad_sch (KiCad schematic)
At the start: 68 parts, among them J2 Conn_01x03_Pin, J4 Conn_01x64_Castellated_Pads, U1 RP2350B_C42415655, U3 ME6217C33M5G, U4 W25Q128JVSIQTR, U5 RPI Radio Module 2, U6 APS6404L-3SQR, X1 ABM8-272-T3_C20625731

Commit message: JLCImport production files, fresh README images, copper parts out of BOM/CPL
- production/: Fabrication Toolkit output and its options file removed;
  JLCImport (jlcimport-cli production) gerbers, BOM, CPL and report
  regenerated from the current board
- TP1-TP5 and J4 (copper only) excluded from the BOM and position files,
  as JP1-JP4 already are, so no blank BOM rows and no bottom-side CPL
  entries (scripts/pico_testpads.py; Castellated_Pad_64 and the Pico
  test-pad footprint carry the same attributes)
- images/: all README renders regenerated (scripts/render-images.sh)
- README: production section describes the JLCImport files
Parts:
- J4, TP1, TP2, TP3, TP4, TP5: now left out of the parts list
Changed lines of the file:
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@@
 		(body_style 1)
 		(exclude_from_sim no)
-		(in_bom yes)
+		(in_bom no)
 		(on_board yes)
-		(in_pos_files yes)
+		(in_pos_files no)
 		(dnp no)
 		(fields_autoplaced yes)
@@
 		(body_style 1)
 		(exclude_from_sim no)
-		(in_bom yes)
+		(in_bom no)
 		(on_board yes)
-		(in_pos_files yes)
+		(in_pos_files no)
 		(dnp no)
 		(fields_autoplaced yes)
@@
 		(body_style 1)
 		(exclude_from_sim no)
-		(in_bom yes)
+		(in_bom no)
 		(on_board yes)
-		(in_pos_files yes)
+		(in_pos_files no)
 		(dnp no)
 		(fields_autoplaced yes)
@@
 		(body_style 1)
 		(exclude_from_sim no)
-		(in_bom yes)
+		(in_bom no)
 		(on_board yes)
-		(in_pos_files yes)
+		(in_pos_files no)
 		(dnp no)
 		(property "Reference" "TP3"
@@
 		(body_style 1)
 		(exclude_from_sim no)
-		(in_bom yes)
+		(in_bom no)
 		(on_board yes)
-		(in_pos_files yes)
+		(in_pos_files no)
 		(dnp no)
 		(property "Reference" "TP4"
@@
 		(body_style 1)
 		(exclude_from_sim no)
-		(in_bom yes)
+		(in_bom no)
 		(on_board yes)
-		(in_pos_files yes)
+		(in_pos_files no)
 		(dnp no)
 		(property "Reference" "TP5"
